File: HW/SBC/pluto.kicad_pcb (KiCad board)
At the start: 2 copper layers, 76 parts, among them J1 VIA1PA, J2 VIA1PB, J3 VIA2PB, J4 BARREL_JACK, J5 AY-IO, J6 RS232a, J7 RS232b, J8 JTAG, P1 IDE0, Q1 DS1813, SW1 RESET, U1 WD65C02PLCC44, U12 LM7805CT, U13 LM386, U14 AY-3-8912, U15 74LS32, U16 74LS139, U17 74HC74, U18 74LS08, U19 74LS574, U2 28C256, U20 74LS574, U21 74HC245, U22 MAX238, U23 SC28L92PLCC44, U3 AS6C62256A, U4 DS1511Y+, U5 WD65C22PLCC44, U6 WD65C22PLCC44, U7 ispMACH4A5, U8 74HC74, X1 8 MHz, X2 3.6864MHz

Commit message: Added CPLD to schematics. Updates rest of schematics to use CPLD
Parts:
- removed C10: 10uF, Capacitors_ThroughHole:CP_Radial_D5.0mm_P2.00mm
- removed C11: 10nF, Capacitors_ThroughHole:C_Disc_D3.8mm_W2.6mm_P2.50mm
- removed C12: 47nF, Capacitors_ThroughHole:C_Disc_D3.8mm_W2.6mm_P2.50mm
- removed C13: 220uF 10V, Capacitors_ThroughHole:CP_Radial_D6.3mm_P2.50mm
- removed C14: 0.1uF, Capacitors_ThroughHole:C_Disc_D4.7mm_W2.5mm_P5.00mm
- removed C7: 100 uF, Capacitors_ThroughHole:CP_Radial_D6.3mm_P2.50mm
- removed C8: 10 uF, Capacitors_ThroughHole:CP_Radial_D5.0mm_P2.00mm
- removed C9: 2.2nF, Capacitors_ThroughHole:C_Disc_D3.8mm_W2.6mm_P2.50mm
- removed LS1: Speaker, Connect:Stereo_Jack_3.5mm_Switch_Ledino_KB3SPRS
- removed R1: 22k, Resistors_ThroughHole:R_Axial_DIN0411_L9.9mm_D3.6mm_P12.70mm_Horizontal
- removed R2: 470, Resistors_ThroughHole:R_Axial_DIN0411_L9.9mm_D3.6mm_P12.70mm_Horizontal
- removed R3: 4.7k, Resistors_ThroughHole:R_Axial_DIN0411_L9.9mm_D3.6mm_P12.70mm_Horizontal
- removed R4, R9: 1k, Resistors_ThroughHole:R_Axial_DIN0411_L9.9mm_D3.6mm_P12.70mm_Horizontal
- removed R5: 10, Resistors_ThroughHole:R_Axial_DIN0411_L9.9mm_D3.6mm_P12.70mm_Horizontal
- removed U12: LM7805CT, TO_SOT_Packages_THT:TO-220-3_Horizontal
- removed U13: LM386, Housings_DIP:DIP-8_W7.62mm_Socket
- removed U14: AY-3-8912, Housings_DIP:DIP-28_W15.24mm_Socket
- removed U15: 74LS32, Housings_DIP:DIP-14_W7.62mm_Socket
- removed U16: 74LS139, Housings_DIP:DIP-16_W7.62mm_Socket
- removed U17: 74HC74, Housings_DIP:DIP-14_W7.62mm_Socket
- removed U18: 74LS08, Housings_DIP:DIP-14_W7.62mm_Socket
- added J9: TEST_2P, Pin_Headers:Pin_Header_Straight_1x02_Pitch2.54mm, F.Cu at (133.3, 21.0)
- J4: value BARREL_JACK -> POWER; footprint Connect:BARREL_JACK -> Connectors_Molex:Molex_NanoFit_1x04x2.50mm_Angled
- J5: value AY-IO -> VIA2PA
- moved MK2 238.3 mm to (20.3, 19.7)
- moved MK3 233.4 mm to (20.3, 125.1)
- moved U2 174.3 mm to (90.2, 20.3)
- moved R8 169.1 mm to (184.8, 21.6), turned to 180 degrees
- moved P1 143.4 mm to (193.0, 79.4), turned to 180 degrees
- moved C3 142.4 mm to (45.1, 29.8), turned to 90 degrees
- moved U4 141.1 mm to (111.8, 20.3)
- moved C15 138.0 mm to (174.6, 109.9), turned to 90 degrees
- moved J8 128.8 mm to (81.3, 66.0)
- moved U19 124.9 mm to (177.2, 27.3)
- moved C19 124.1 mm to (174.6, 104.8), turned to 90 degrees
- moved C5 122.5 mm to (123.2, 22.9), turned to 270 degrees
- moved J5 122.3 mm to (84.5, 123.8), turned to 90 degrees
- moved MK5 119.7 mm to (136.5, 125.1)
- moved C17 118.8 mm to (161.3, 109.9), turned to 270 degrees
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Connections:
- net /16bit IDE interface/CLK renamed /Address decoding and support section/CLK
- J4 pad 1: +9V -> (no net)
- J5 pad 10: /Audio/IO_A5 -> Net-(J5-Pad10)
- J5 pad 11: /Audio/IO_A6 -> Net-(J5-Pad11)
- J5 pad 12: /Audio/IO_A7 -> Net-(J5-Pad12)
- J5 pad 3: (no net) -> Net-(J5-Pad3)
- J5 pad 4: (no net) -> Net-(J5-Pad4)
- J5 pad 5: /Audio/IO_A0 -> Net-(J5-Pad5)
- J5 pad 6: /Audio/IO_A1 -> Net-(J5-Pad6)
- J5 pad 7: /Audio/IO_A2 -> Net-(J5-Pad7)
- J5 pad 8: /Audio/IO_A3 -> Net-(J5-Pad8)
- J5 pad 9: /Audio/IO_A4 -> Net-(J5-Pad9)
- P1 pad 23: /16bit IDE interface/~DIOW -> /16bit IDE interface/DIOW
- P1 pad 25: /16bit IDE interface/~DIOR -> /16bit IDE interface/DIOR
- P1 pad 37: /16bit IDE interface/~IDE:CS0 -> /16bit IDE interface/IDE_CS0
- U1 pad 14: /16bit IDE interface/A3 -> /Address decoding and support section/A3
- U19 pad 1: Net-(U16-Pad4) -> /16bit IDE interface/FROM_OE
- U19 pad 11: Net-(U16-Pad5) -> /16bit IDE interface/FROM_CLK
- U2 pad 22: /16bit IDE interface/~MRD -> /Address decoding and support section/~MRD
- U2 pad 7: /16bit IDE interface/A3 -> /Address decoding and support section/A3
- U20 pad 1: Net-(U15-Pad9) -> /16bit IDE interface/TO_OE
- U20 pad 11: Net-(U16-Pad11) -> /16bit IDE interface/TO_CLK
- U21 pad 1: /16bit IDE interface/~DIOR -> /16bit IDE interface/OBT_DIR
- U21 pad 19: Net-(U18-Pad3) -> /16bit IDE interface/OBT_OE
- U23 pad 10: /16bit IDE interface/~MRD -> /Address decoding and support section/~MRD
- U23 pad 7: /16bit IDE interface/A3 -> /Address decoding and support section/A3
- U23 pad 9: /16bit IDE interface/~MWR -> /Address decoding and support section/~MWR
- U3 pad 22: /16bit IDE interface/~MRD -> /Address decoding and support section/~MRD
- U3 pad 27: /16bit IDE interface/~MWR -> /Address decoding and support section/~MWR
- U3 pad 7: /16bit IDE interface/A3 -> /Address decoding and support section/A3
- U4 pad 22: /16bit IDE interface/~MRD -> /Address decoding and support section/~MRD
- U4 pad 27: /16bit IDE interface/~MWR -> /Address decoding and support section/~MWR
- U4 pad 7: /16bit IDE interface/A3 -> /Address decoding and support section/A3
- U5 pad 39: /16bit IDE interface/A3 -> /Address decoding and support section/A3
- U6 pad 2: /Audio/V2PA0 -> Net-(J5-Pad3)
- U6 pad 3: /Audio/V2PA1 -> Net-(J5-Pad4)
- U6 pad 39: /16bit IDE interface/A3 -> /Address decoding and support section/A3
- U6 pad 4: /Audio/V2PA2 -> Net-(J5-Pad5)
- U6 pad 43: /Audio/V2CA2 -> Net-(J5-Pad12)
- U6 pad 44: /Audio/V2CA1 -> Net-(J5-Pad11)
- U6 pad 5: /Audio/V2PA3 -> Net-(J5-Pad6)
- U6 pad 6: /Audio/V2PA4 -> Net-(J5-Pad7)
- U6 pad 7: /Audio/V2PA5 -> Net-(J5-Pad8)
- U6 pad 8: /Audio/V2PA6 -> Net-(J5-Pad9)
- U6 pad 9: /Audio/V2PA7 -> Net-(J5-Pad10)
- U7 pad 14: /Address decoding and support section/A9 -> /Address decoding and support section/A13
- U7 pad 15: /Address decoding and support section/A8 -> /Address decoding and support section/~RAMSEL
- U7 pad 16: /Address decoding and support section/A7 -> /Address decoding and support section/A12
- U7 pad 17: /Address decoding and support section/A6 -> /16bit IDE interface/FROM_CLK
- U7 pad 18: /Address decoding and support section/A5 -> /Address decoding and support section/A11
- U7 pad 19: /16bit IDE interface/~7F6X -> /16bit IDE interface/IDE_CS0
- U7 pad 2: /16bit IDE interface/~MWR -> /Address decoding and support section/~7FAX
- U7 pad 20: /Address decoding and support section/R/~W -> /16bit IDE interface/OBT_OE
- U7 pad 24: /Address decoding and support section/~7F8X -> /16bit IDE interface/FROM_OE
- U7 pad 25: /16bit IDE interface/~RES -> /16bit IDE interface/DIOW
- U7 pad 26: /Address decoding and support section/~7FCX -> /16bit IDE interface/TO_OE
- U7 pad 27: (no net) -> /Address decoding and support section/A10
- U7 pad 28: (no net) -> /16bit IDE interface/OBT_DIR
- U7 pad 29: Net-(U7-Pad29) -> /Address decoding and support section/A9
- U7 pad 3: /Address decoding and support section/A14 -> /Address decoding and support section/~7FEX
- U7 pad 30: /Address decoding and support section/~7FEX -> /16bit IDE interface/TO_CLK
- U7 pad 31: (no net) -> /Address decoding and support section/A8
- U7 pad 36: (no net) -> /Address decoding and support section/A7
- U7 pad 37: (no net) -> /Address decoding and support section/RES
- U7 pad 38: (no net) -> /Address decoding and support section/A6
- U7 pad 39: Net-(U7-Pad39) -> /16bit IDE interface/DIOR
- U7 pad 4: /16bit IDE interface/~MRD -> (no net)
- U7 pad 40: Net-(U7-Pad40) -> /Address decoding and support section/A5
- U7 pad 41: /Address decoding and support section/~7FAX -> /Address decoding and support section/~MRD
- U7 pad 42: (no net) -> /16bit IDE interface/~RES
- U7 pad 43: /Address decoding and support section/~RAMSEL -> /Address decoding and support section/~MWR
- U7 pad 5: /Address decoding and support section/A13 -> /Address decoding and support section/A3
- U7 pad 6: /Address decoding and support section/A12 -> /Address decoding and support section/~7F8X
- U7 pad 7: /Address decoding and support section/A11 -> /Address decoding and support section/R/~W
- U7 pad 8: /Address decoding and support section/RES -> /Address decoding and support section/~7FCX
- U7 pad 9: /Address decoding and support section/A10 -> /Address decoding and support section/A14
Routing:
- added copper zone on GND.Cu, net GND
- added copper zone on VCC.Cu, net VCC
Other:
- board outline added: 181.6 x 113 mm
- copper layers 2 -> 4
- net class GND added: clearance 0.2, trace_width 0.25, via_dia 0.6, via_drill 0.4
- net class VCC added: clearance 0.2, trace_width 0.45, via_dia 0.6, via_drill 0.4
