File: SBC/address_decoding_and_support.sch (KiCad schematic (older format))
At the start: 9 parts, among them Q1 DS1813, SW1 RESET, U7 ispMACH4A5, U8 74HC74, X1 8 MHz

Commit message: Board ready for production. Added a reset IC that does both low and high logic RES. A power switch and fuse holder is in place. The expansion bus is back, but with an IDC 40 pin connector.
Parts:
- removed Q1: DS1813, TO_SOT_Packages_THT:TO-92_Inline_Narrow_Oval, symbol Q_NPN_EBC
- added C4: 15uF, Capacitors_ThroughHole:CP_Radial_Tantal_D4.5mm_P2.50mm, symbol CP_Small
- added C6: 0.1uF, Capacitors_ThroughHole:C_Disc_D4.7mm_W2.5mm_P5.00mm, symbol C_Small
- added R2: 22k, Resistors_ThroughHole:R_Axial_DIN0411_L9.9mm_D3.6mm_P7.62mm_Vertical, symbol R_Small
- added R3: 475, Resistors_ThroughHole:R_Axial_DIN0411_L9.9mm_D3.6mm_P7.62mm_Vertical, symbol R_Small
- added R4: 3.3k, Resistors_ThroughHole:R_Axial_DIN0411_L9.9mm_D3.6mm_P7.62mm_Vertical, symbol R_Small
- added U5: TL7705B, Housings_DIP:DIP-8_W7.62mm_Socket, symbol TL7705B
Connections:
- net labels removed: RESET
- wire segments 95 -> 106
- no-connect marks 6 -> 8
Other:
- moved on the sheet: C21, C22, RN2, SW1, U7
