File: SBC/address_decoding_and_support.sch (KiCad schematic (older format))
At the start: 14 parts, among them SW1 RESET, U5 TL7705B, U7 ispMACH4A5, U8 74HC74, X1 8 MHz

Commit message: KiCad updated schematics
Parts:
- C21, C22, C6: symbol device:C_Small -> pluto-rescue:C_Small-device
- C4: symbol device:CP_Small -> pluto-rescue:CP_Small-device
- R2, R3, R4: symbol device:R_Small -> pluto-rescue:R_Small-device
- RN1, RN2: symbol device:R_Network07 -> pluto-rescue:R_Network07-device
- SW1: symbol switches:SW_Push -> pluto-rescue:SW_Push-switches
- X1: symbol Oscillators:CXO_DIP8 -> pluto-rescue:CXO_DIP8-Oscillators
Changed lines of the file:
@@
 EESchema Schematic File Version 4
 LIBS:pluto-cache
-EELAYER 29 0
+EELAYER 30 0
 EELAYER END
 $Descr A4 11693 8268
@@
 $EndDescr
 $Comp
-L device:R_Network07 RN2
+L pluto-rescue:R_Network07-device RN2
 U 1 1 58D6C524
 P 3950 1400
@@
 $EndComp
 $Comp
-L Oscillators:CXO_DIP8 X1
+L pluto-rescue:CXO_DIP8-Oscillators X1
 U 1 1 58D6C921
 P 4350 6450
@@
 $EndComp
 $Comp
-L switches:SW_Push SW1
+L pluto-rescue:SW_Push-switches SW1
 U 1 1 58D6D3A4
 P 1650 3650
@@
 ~KS
 $Comp
-L device:R_Network07 RN1
+L pluto-rescue:R_Network07-device RN1
 U 1 1 594C05A8
 P 1350 6000
@@
 $EndComp
 $Comp
-L device:C_Small C22
+L pluto-rescue:C_Small-device C22
 U 1 1 59F44526
 P 9375 4350
@@
 $EndComp
 $Comp
-L device:C_Small C21
+L pluto-rescue:C_Small-device C21
 U 1 1 59F44553
 P 8175 4350
@@
 $EndComp
 $Comp
-L device:R_Small R2
+L pluto-rescue:R_Small-device R2
 U 1 1 5A37C778
 P 1650 2975
@@
 $EndComp
 $Comp
-L device:R_Small R3
+L pluto-rescue:R_Small-device R3
 U 1 1 5A37C7D7
 P 2050 3700
@@
 RES
 $Comp
-L device:CP_Small C4
+L pluto-rescue:CP_Small-device C4
 U 1 1 5A37EF31
 P 2050 4025
@@
 $EndComp
 $Comp
-L device:C_Small C6
+L pluto-rescue:C_Small-device C6
 U 1 1 5A37FB89
 P 3650 3625
@@
 NoConn ~ 9425 2150
 $Comp
-L device:R_Small R4
+L pluto-rescue:R_Small-device R4
 U 1 1 5A3880A9
 P 3950 3475
