File: SBC/power_and_expansion.sch (KiCad schematic (older format))
At the start: 9 parts, among them J4 POWER, J8 JTAG, J9 TEST_2P

Commit message: Board ready for production. Added a reset IC that does both low and high logic RES. A power switch and fuse holder is in place. The expansion bus is back, but with an IDC 40 pin connector.
Parts:
- removed J9: TEST_2P, Pin_Headers:Pin_Header_Straight_1x02_Pitch2.54mm, symbol TEST_2P
- added D1: LED, LEDs:LED_D3.0mm, symbol LED
- added F1: 1Amp, Fuse_Holders_and_Fuses:Fuseholder5x20_horiz_open_Schurter_0031_8201, symbol Fuse_Small
- added J1: VCC1, Pin_Headers:Pin_Header_Straight_1x01_Pitch2.54mm, symbol TEST_1P
- added J10: GND3, Pin_Headers:Pin_Header_Straight_1x01_Pitch2.54mm, symbol TEST_1P
- added J11: Expansion Bus, Connectors_IDC:IDC-Header_2x20_Pitch2.54mm_Straight, symbol Conn_02x20_Odd_Even
- added J2: GND1, Pin_Headers:Pin_Header_Straight_1x01_Pitch2.54mm, symbol TEST_1P
- added J3: VCC2, Pin_Headers:Pin_Header_Straight_1x01_Pitch2.54mm, symbol TEST_1P
- added J5: GND2, Pin_Headers:Pin_Header_Straight_1x01_Pitch2.54mm, symbol TEST_1P
- added J9: VCC3, Pin_Headers:Pin_Header_Straight_1x01_Pitch2.54mm, symbol TEST_1P
- added R1: 1kOhm, Resistors_ThroughHole:R_Axial_DIN0411_L9.9mm_D3.6mm_P12.70mm_Horizontal, symbol R_Small
- added S1: SPDT, Switches_THT:SW-SPDT-0900766b81587629, symbol SPDT
Connections:
- net labels added: A0, A1, A10, A11, A12, A13, A14, A15, A2, A3, A4, A5, A6, A7, A8, A9, A[0..15], CLK, D0, D1, D2, D3, D4, D5, D6, D7, D[0..7], PWR_IN, R/~W, RDY, ~7FAX, ~7FCX, ~IRQ, ~MRD, ~MWR, ~NMI, ~RES
- wire segments 13 -> 59
- no-connect marks 3 -> 6
Other:
- moved on the sheet: J4, J8
