File: SBC/power_and_expansion.sch (KiCad schematic (older format))
At the start: 19 parts, among them J1 VCC1, J10 GND3, J11 Expansion Bus, J2 GND1, J3 VCC2, J4 POWER, J5 GND2, J8 JTAG, J9 VCC3

Commit message: KiCad updated schematics
Parts:
- F1: symbol device:Fuse_Small -> pluto-rescue:Fuse_Small-device
- J1, J10, J2, J3, J5, J9: symbol conn:TEST_1P -> pluto-rescue:TEST_1P-conn
- J4: symbol conn:CONN_01X04 -> pluto-rescue:CONN_01X04-conn
- J8: symbol conn:CONN_02X05 -> pluto-rescue:CONN_02X05-conn
- MK1, MK2, MK3, MK4, MK5, MK6: symbol mechanical:Mounting_Hole -> pluto-rescue:Mounting_Hole-mechanical
- R1: symbol device:R_Small -> pluto-rescue:R_Small-device
- S1: symbol standard:SPDT -> pluto-rescue:SPDT-standard
Changed lines of the file:
@@
 EESchema Schematic File Version 4
 LIBS:pluto-cache
-EELAYER 29 0
+EELAYER 30 0
 EELAYER END
 $Descr A4 11693 8268
@@
 $EndDescr
 $Comp
-L mechanical:Mounting_Hole MK2
+L pluto-rescue:Mounting_Hole-mechanical MK2
 U 1 1 59149E60
 P 1825 3025
@@
 $EndComp
 $Comp
-L mechanical:Mounting_Hole MK3
+L pluto-rescue:Mounting_Hole-mechanical MK3
 U 1 1 59149E83
 P 1825 3450
@@
 $EndComp
 $Comp
-L mechanical:Mounting_Hole MK1
+L pluto-rescue:Mounting_Hole-mechanical MK1
 U 1 1 5932DD04
 P 1125 3950
@@
 $EndComp
 $Comp
-L mechanical:Mounting_Hole MK4
+L pluto-rescue:Mounting_Hole-mechanical MK4
 U 1 1 5932DD62
 P 1825 3950
@@
 $EndComp
 $Comp
-L conn:CONN_02X05 J8
+L pluto-rescue:CONN_02X05-conn J8
 U 1 1 59F22BEE
 P 4275 3000
@@
 NoConn ~ 4025 3200
 $Comp
-L mechanical:Mounting_Hole MK5
+L pluto-rescue:Mounting_Hole-mechanical MK5
 U 1 1 59F424EE
 P 2600 3000
@@
 $EndComp
 $Comp
-L mechanical:Mounting_Hole MK6
+L pluto-rescue:Mounting_Hole-mechanical MK6
 U 1 1 59F42548
 P 2600 3350
@@
 $EndComp
 $Comp
-L conn:CONN_01X04 J4
+L pluto-rescue:CONN_01X04-conn J4
 U 1 1 5A1609CD
 P 7650 1725
@@
 Connection ~ 7375 1675
 $Comp
-L device:Fuse_Small F1
+L pluto-rescue:Fuse_Small-device F1
 U 1 1 5A30BB96
 P 6800 1575
@@
 $EndComp
 $Comp
-L standard:SPDT S1
+L pluto-rescue:SPDT-standard S1
 U 1 1 5A30BD5A
 P 6425 1625
@@
 $EndComp
 $Comp
-L device:R_Small R1
+L pluto-rescue:R_Small-device R1
 U 1 1 5A30C649
 P 5625 1625
@@
 	5425 1625 5525 1625
 $Comp
-L conn:TEST_1P J1
+L pluto-rescue:TEST_1P-conn J1
 U 1 1 5A30C731
 P 1450 5025
@@
 $EndComp
 $Comp
-L conn:TEST_1P J3
+L pluto-rescue:TEST_1P-conn J3
 U 1 1 5A30C776
 P 1775 5025
@@
 $EndComp
 $Comp
-L conn:TEST_1P J9
+L pluto-rescue:TEST_1P-conn J9
 U 1 1 5A30C7BB
 P 2125 5025
@@
 $EndComp
 $Comp
-L conn:TEST_1P J2
+L pluto-rescue:TEST_1P-conn J2
 U 1 1 5A30C814
 P 1450 5625
@@
 $EndComp
 $Comp
-L conn:TEST_1P J5
+L pluto-rescue:TEST_1P-conn J5
 U 1 1 5A30C853
 P 1775 5625
@@
 $EndComp
 $Comp
-L conn:TEST_1P J10
+L pluto-rescue:TEST_1P-conn J10
 U 1 1 5A30C89C
 P 2125 5625
