File: SBC/via_rtc.sch (KiCad schematic (older format))
At the start: 12 parts, among them J1 VIA1PA, J2 VIA1PB, J3 VIA2PB, J5 VIA2PA, U4 DS1511Y+, U5 WD65C22PLCC44, U6 WD65C22PLCC44

Commit message: Board ready for production. Added a reset IC that does both low and high logic RES. A power switch and fuse holder is in place. The expansion bus is back, but with an IDC 40 pin connector.
Parts:
- removed C4, C6: 0.1uF, Capacitors_ThroughHole:C_Disc_D4.7mm_W2.5mm_P5.00mm, symbol C
- removed D1, D2: D, Diodes_ThroughHole:D_DO-35_SOD27_P7.62mm_Horizontal, symbol D_Small
- removed J1: VIA1PA, Connectors_IDC:IDC-Header_2x07_Pitch2.54mm_Straight, symbol CONN_02X07
- removed J2: VIA1PB, Connectors_IDC:IDC-Header_2x07_Pitch2.54mm_Straight, symbol CONN_02X07
- removed J3: VIA2PB, Connectors_IDC:IDC-Header_2x07_Pitch2.54mm_Straight, symbol CONN_02X07
- removed J5: VIA2PA, Connectors_IDC:IDC-Header_2x07_Pitch2.54mm_Straight, symbol CONN_02X07
- removed U5, U6: WD65C22PLCC44, Housings_LCC:PLCC-44_THT-Socket, symbol WD65C22PLCC44
Connections:
- net labels removed: CLK, R/~W, ~7FAX, ~7FCX
- wire segments 175 -> 27
Other:
- moved on the sheet: C5, U4
