File: SBC/via_rtc.sch (KiCad schematic (older format))
At the start: 2 parts, among them U4 DS1511Y+

Commit message: Small changes to schematics
Parts:
- C5: symbol C -> pluto-rescue:C
- U4: symbol DS1511Y+ -> saturn:DS1511Y+
