File: SBC/IDE16bit.sch (KiCad schematic (older format))
At the start: 8 parts, among them P1 IDE0, U19 74LS574, U20 74LS574, U21 74HC245

Commit message: Small changes to schematics
Parts:
- D3: symbol LED -> pluto-rescue:LED
- P1: symbol CONN_02X20 -> conn:CONN_02X20
- R6, R7, R8: symbol R -> pluto-rescue:R
- U19, U20: symbol 74LS574 -> pluto-rescue:74LS574
- U21: symbol 74HC245 -> pluto-rescue:74HC245
Connections:
- wire segments 102 -> 108
