File: SBC/IDE16bit.sch (KiCad schematic (older format))
At the start: 8 parts, among them P1 IDE0, U19 74LS574, U20 74LS574, U21 74HC245

Commit message: KiCad updated schematics
Parts:
- P1: symbol conn:CONN_02X20 -> pluto-rescue:CONN_02X20-conn
Changed lines of the file:
@@
 EESchema Schematic File Version 4
 LIBS:pluto-cache
-EELAYER 29 0
+EELAYER 30 0
 EELAYER END
 $Descr A3 16535 11693
@@
 D7
 $Comp
-L conn:CONN_02X20 P1
+L pluto-rescue:CONN_02X20-conn P1
 U 1 1 5932FB36
 P 10300 2825
