File: SBC/cpu_rom_ram.sch (KiCad schematic (older format))
At the start: 6 parts, among them U1 WD65C02PLCC44, U2 28C256, U3 AS6C62256A

Commit message: Small changes to schematics
Parts:
- C1, C2, C3: symbol C -> pluto-rescue:C
- U1: symbol WD65C02PLCC44 -> 65xx:WD65C02PLCC44
- U2: symbol 28C256-RESCUE-pluto -> pluto-rescue:28C256-RESCUE-pluto
- U3: symbol AS6C62256A -> pluto:AS6C62256A
