File: SBC/cpu_rom_ram.sch (KiCad schematic (older format))
At the start: 6 parts, among them U1 WD65C02PLCC44, U2 28C256, U3 AS6C62256A

Commit message: KiCad updated schematics
Parts:
- U1: symbol 65xx:WD65C02PLCC44 -> pluto-rescue:WD65C02PLCC44-65xx
Changed lines of the file:
@@
 EESchema Schematic File Version 4
 LIBS:pluto-cache
-EELAYER 29 0
+EELAYER 30 0
 EELAYER END
 $Descr A4 11693 8268
@@
 ~SO
 $Comp
-L 65xx:WD65C02PLCC44 U1
+L pluto-rescue:WD65C02PLCC44-65xx U1
 U 1 1 59EBAA82
 P 2175 2600
