File: SBC/duart_rs232.sch (KiCad schematic (older format))
At the start: 11 parts, among them J6 RS232a, J7 RS232b, U22 MAX238, U23 SC28L92PLCC44, X2 3.6864MHz

Commit message: Small changes to schematics
Parts:
- C15, C16, C17, C18, C19: symbol CP1_Small -> device:CP1_Small
- C20: symbol C_Small -> device:C_Small
- J6, J7: symbol CONN_02X05 -> conn:CONN_02X05
- U22: symbol MAX238 -> pluto:MAX238
- U23: symbol SC28L92PLCC44 -> pluto:SC28L92PLCC44
- X2: symbol CXO_DIP8 -> Oscillators:CXO_DIP8
