File: SBC/duart_rs232.sch (KiCad schematic (older format))
At the start: 11 parts, among them J6 RS232a, J7 RS232b, U22 MAX238, U23 SC28L92PLCC44, X2 3.6864MHz

Commit message: KiCad updated schematics
Parts:
- C15, C16, C17, C18, C19: symbol device:CP1_Small -> pluto-rescue:CP1_Small-device
- C20: symbol device:C_Small -> pluto-rescue:C_Small-device
- J6, J7: symbol conn:CONN_02X05 -> pluto-rescue:CONN_02X05-conn
- X2: symbol Oscillators:CXO_DIP8 -> pluto-rescue:CXO_DIP8-Oscillators
Changed lines of the file:
@@
 EESchema Schematic File Version 4
 LIBS:pluto-cache
-EELAYER 29 0
+EELAYER 30 0
 EELAYER END
 $Descr A4 11693 8268
@@
 $EndComp
 $Comp
-L conn:CONN_02X05 J6
+L pluto-rescue:CONN_02X05-conn J6
 U 1 1 59ECCE48
 P 1500 2750
@@
 $EndComp
 $Comp
-L conn:CONN_02X05 J7
+L pluto-rescue:CONN_02X05-conn J7
 U 1 1 59ECCF01
 P 1500 3475
@@
 $EndComp
 $Comp
-L device:CP1_Small C18
+L pluto-rescue:CP1_Small-device C18
 U 1 1 59ECCF2A
 P 4650 1575
@@
 $EndComp
 $Comp
-L device:CP1_Small C19
+L pluto-rescue:CP1_Small-device C19
 U 1 1 59ECCF53
 P 4650 1975
@@
 $EndComp
 $Comp
-L device:CP1_Small C15
+L pluto-rescue:CP1_Small-device C15
 U 1 1 59ECCF86
 P 2750 1250
@@
 $EndComp
 $Comp
-L device:CP1_Small C16
+L pluto-rescue:CP1_Small-device C16
 U 1 1 59ECCFE5
 P 2750 1775
@@
 $EndComp
 $Comp
-L device:CP1_Small C17
+L pluto-rescue:CP1_Small-device C17
 U 1 1 59ECD006
 P 4325 1150
@@
 A[0..15]
 $Comp
-L device:C_Small C20
+L pluto-rescue:C_Small-device C20
 U 1 1 59ED58A6
 P 7475 5525
@@
 NoConn ~ 7650 5000
 $Comp
-L Oscillators:CXO_DIP8 X2
+L pluto-rescue:CXO_DIP8-Oscillators X2
 U 1 1 59EDF126
 P 9675 4875
