File: SBC/pluto.sch (KiCad schematic (older format))
At the start: 0 parts

Commit message: Preparation for Pluto v3.0
Changed lines of the file:
@@
 EESchema Schematic File Version 4
 LIBS:pluto-cache
-EELAYER 29 0
+EELAYER 30 0
 EELAYER END
 $Descr A4 11693 8268
@@
 F5 "BE" I R 3225 2250 60
 F6 "~IRQ" I L 1350 2050 60
-F7 "R/~W" O L 1350 1850 60
+F7 "R-~W" O L 1350 1850 60
 F8 "~NMI" I R 3225 1750 60
 F9 "CLK" I R 3225 2500 60
@@
 F7 "~MWR" I L 7025 1100 60
 F8 "~MRD" I L 7025 1000 60
-F9 "~7F8X" I L 7025 1225 60
-F10 "~KS" I L 7025 2125 60
+F9 "~KS" I L 7025 2125 60
+F10 "~RTC" I L 7025 1225 60
 $EndSheet
 $Sheet
@@
 F1 "address_decoding_and_support.sch" 60
 F2 "CLK" O R 5900 1750 60
-F3 "A[0..15]" I R 5900 3275 60
-F4 "~MRD" O R 5900 1000 60
-F5 "~MWR" O R 5900 1100 60
-F6 "~ROMSEL" O L 3825 1325 60
-F7 "~RAMSEL" O L 3825 1450 60
-F8 "R/~W" I R 5900 1875 60
-F9 "~IRQ" B R 5900 2000 60
-F10 "~NMI" O L 3825 1750 60
-F11 "BE" O L 3825 2250 60
-F12 "~PWR" O R 5900 1625 60
-F13 "RDY" O L 3825 1200 60
-F14 "~RES" O L 3825 2400 60
-F15 "~7F8X" O R 5900 1225 60
-F16 "~7FEX" O L 3825 3275 60
-F17 "~KS" O R 5900 2125 60
-F18 "~SO" O L 3825 1975 60
-F19 "RES" O L 3825 2575 60
-F20 "TDI" I R 5900 2250 60
-F21 "TDO" O R 5900 2350 60
-F22 "TCK" I R 5900 2450 60
-F23 "TMS" I R 5900 2550 60
-F24 "FROM_OE" O R 5900 3075 60
-F25 "FROM_CLK" O L 3825 3000 60
-F26 "TO_OE" O R 5900 3175 60
-F27 "TO_CLK" O L 3825 2900 60
-F28 "OBT_OE" O L 3825 2800 60
-F29 "OBT_DIR" O L 3825 2700 60
-F30 "DIOR" O R 5900 2875 60
-F31 "DIOW" O R 5900 2975 60
-F32 "IDE_CS0" O R 5900 2775 60
-F33 "~7FAX" O R 5900 1325 60
-F34 "~7FCX" O R 5900 1450 60
+F3 "~IRQ" B R 5900 2000 60
+F4 "~NMI" O L 3825 1750 60
+F5 "BE" O L 3825 2250 60
+F6 "~PWR" O R 5900 1625 60
+F7 "RDY" O L 3825 1200 60
+F8 "~RES" O L 3825 2400 60
+F9 "~KS" O R 5900 2125 60
+F10 "~SO" O L 3825 1975 60
+F11 "RES" O L 3825 2575 60
+F12 "A[0..15]" I R 5900 3275 60
+F13 "R-~W" I R 5900 1875 60
+F14 "~MRD" O L 3825 1000 60
+F15 "~MWR" O L 3825 1100 60
+F16 "~RAMSEL" O L 3825 1450 60
+F17 "~ROMSEL" O L 3825 1325 60
+F18 "~DUART" O L 3825 3275 60
+F19 "~VIA1SEL" O L 3825 2775 60
+F20 "~VIA2SEL" O L 3825 2925 60
+F21 "~RTC" O R 5900 1225 60
+F22 "~IO" O R 5900 2975 60
 $EndSheet
 $Sheet
@@
 F0 "Power and mounting holes" 60
 F1 "power_and_expansion.sch" 60
-F2 "TDI" O L 7575 4000 60
-F3 "TDO" I L 7575 4100 60
-F4 "TCK" O L 7575 4200 60
-F5 "TMS" O L 7575 4300 60
-F6 "~7FAX" I R 9625 4550 60
-F7 "~7FCX" I R 9625 4425 60
-F8 "~IRQ" O L 7575 4700 60
-F9 "~RES" O R 9625 5100 60
-F10 "~MRD" I L 7575 4825 60
-F11 "~MWR" I L 7575 4950 60
-F12 "R/~W" I L 7575 4575 60
-F13 "CLK" I L 7575 4450 60
-F14 "~NMI" I R 9625 4900 60
-F15 "RDY" I R 9625 5300 60
-F16 "D[0..7]" B R 9625 3950 60
-F17 "A[0..15]" I R 9625 4075 60
+F2 "~IRQ" O L 7575 4700 60
+F3 "~RES" O R 9625 5100 60
+F4 "~MRD" I L 7575 4825 60
+F5 "~MWR" I L 7575 4950 60
+F6 "R/~W" I L 7575 4575 60
+F7 "CLK" I L 7575 4450 60
+F8 "~NMI" I R 9625 4900 60
+F9 "RDY" I R 9625 5300 60
+F10 "D[0..7]" B R 9625 3950 60
+F11 "A[0..15]" I R 9625 4075 60
+F12 "~IO" O L 7575 5100 60
 $EndSheet
 $Sheet
@@
 F4 "A[0..15]" I R 5900 5575 60
 F5 "~IRQ" O R 5900 4750 60
-F6 "TO_OE" I R 5900 4875 60
-F7 "TO_CLK" I L 3750 4250 60
-F8 "FROM_CLK" I L 3750 4150 60
-F9 "FROM_OE" I R 5900 5000 60
-F10 "OBT_DIR" I L 3750 4450 60
-F11 "OBT_OE" I L 3750 4350 60
-F12 "IDE_CS0" I R 5900 4175 60
-F13 "DIOR" I R 5900 4075 60
-F14 "DIOW" I R 5900 3975 60
+F6 "R-~W" I R 5900 4875 60
+F7 "CLK" I L 3750 4325 60
+F8 "~VIA2SEL" I L 3750 4575 60
+F9 "~VIA1SEL" I L 3750 4900 60
 $EndSheet
 Text Label 975  2375 0    60   ~ 0
@@
 F6 "~MWR" I L 1325 3525 60
 F7 "~IRQ" O L 1325 3350 60
-F8 "~7FEX" I R 2700 3275 60
+F8 "~DUART" I R 2700 3275 60
 $EndSheet
 Wire Wire Line
@@
 	3225 2500 3325 2500
 Wire Wire Line
-	3325 2500 3325 6025
+	3325 2500 3325 4325
 Wire Wire Line
 	3225 2400 3425 2400
@@
 	750  6350 6400 6350
 Wire Wire Line
-	6400 6350 6400 1875
+	6400 6350 6400 4875
 Wire Wire Line
 	6100 6025 3325 6025
@@
 	3525 3075 2700 3075
 Wire Wire Line
-	5900 3175 6500 3175
-Wire Wire Line
-	6500 3175 6500 4875
-Wire Wire Line
-	6500 4875 5900 4875
-Wire Wire Line
-	5900 3075 6600 3075
-Wire Wire Line
-	6600 3075 6600 5000
-Wire Wire Line
-	6600 5000 5900 5000
-Wire Wire Line
-	3825 3000 3700 3000
-Wire Wire Line
-	3700 3000 3700 4150
-Wire Wire Line
-	3700 4150 3750 4150
-Wire Wire Line
-	3825 2900 3675 2900
-Wire Wire Line
-	3675 2900 3675 4250
-Wire Wire Line
-	3675 4250 3750 4250
-Wire Wire Line
-	3825 2800 3650 2800
-Wire Wire Line
-	3650 2800 3650 4350
-Wire Wire Line
-	3650 4350 3750 4350
-Wire Wire Line
-	3825 2700 3625 2700
-Wire Wire Line
-	3625 2700 3625 4450
-Wire Wire Line
-	3625 4450 3750 4450
+	6400 4875 5900 4875
 Wire Wire Line
 	6125 650  6125 1000
@@
 	6025 775  6025 1100
 Wire Wire Line
-	5900 2975 5950 2975
-Wire Wire Line
-	5950 2975 5950 3975
-Wire Wire Line
-	5950 3975 5900 3975
-Wire Wire Line
-	5900 2875 5975 2875
-Wire Wire Line
-	5975 2875 5975 4075
-Wire Wire Line
-	5975 4075 5900 4075
-Wire Wire Line
-	5900 2775 6000 2775
-Wire Wire Line
-	6000 2775 6000 4175
-Wire Wire Line
-	6000 4175 5900 4175
-Wire Wire Line
 	9650 3550 9650 2500
 Wire Wire Line
@@
 Wire Wire Line
 	5900 1875 6400 1875
-Wire Wire Line
-	5900 1450 6925 1450
-Wire Wire Line
-	5900 1325 6900 1325
-Wire Wire Line
-	5900 2550 6925 2550
-Wire Wire Line
-	6925 2550 6925 4300
-Wire Wire Line
-	6925 4300 7575 4300
-Wire Wire Line
-	7575 4200 6950 4200
-Wire Wire Line
-	6950 4200 6950 2450
-Wire Wire Line
-	6950 2450 5900 2450
-Wire Wire Line
-	5900 2350 6975 2350
-Wire Wire Line
-	6975 2350 6975 4100
-Wire Wire Line
-	6975 4100 7575 4100
-Wire Wire Line
-	7000 4000 7575 4000
-Wire Wire Line
-	7000 2250 7000 4000
-Wire Wire Line
-	7000 2250 5900 2250
 Wire Bus Line
 	9625 3950 10150 3950
@@
 Connection ~ 10150 3950
 Wire Wire Line
-	6925 1450 6925 750
-Wire Wire Line
-	6925 750  9725 750
-Wire Wire Line
-	9725 750  9725 4425
-Wire Wire Line
-	9725 4425 9625 4425
-Wire Wire Line
-	6900 1325 6900 700
-Wire Wire Line
-	6900 700  9775 700
-Wire Wire Line
-	9775 700  9775 4550
-Wire Wire Line
-	9775 4550 9625 4550
-Wire Wire Line
 	6900 1750 6900 4450
 Wire Wire Line
@@
 Wire Wire Line
 	3625 1200 3825 1200
+Wire Wire Line
+	3750 4325 3325 4325
+Connection ~ 3325 4325
+Wire Wire Line
+	3325 4325 3325 6025
+Connection ~ 6400 4875
+Wire Wire Line
+	6400 4875 6400 1875
+Wire Wire Line
+	3825 1000 3425 1000
+Connection ~ 3425 1000
+Wire Wire Line
+	3825 1100 3550 1100
+Connection ~ 3550 1100
+Wire Wire Line
+	7575 5100 6675 5100
+Wire Wire Line
+	6675 5100 6675 2975
+Wire Wire Line
+	6675 2975 5900 2975
+Wire Wire Line
+	3825 2925 3675 2925
+Wire Wire Line
+	3675 2925 3675 4575
+Wire Wire Line
+	3675 4575 3750 4575
+Wire Wire Line
+	3825 2775 3600 2775
+Wire Wire Line
+	3600 2775 3600 4900
+Wire Wire Line
+	3600 4900 3750 4900
 $EndSCHEMATC
