File: HW/address_decoding_and_support.sch (KiCad schematic (older format))
At the start: 16 parts, among them Q1 DS1813, SW1 RESET, SW2 PANIC, U5 TL7705B, U6 PlutoDecoder, U8 74HC74, X1 16MHz

Commit message: Disable power down. Align init code to force a page break when reading the init table.
Parts:
- X1: symbol Oscillator:SG-8002CA -> pluto-rescue:SG-8002CA-Oscillator
Changed lines of the file:
@@
 EESchema Schematic File Version 4
-LIBS:pluto-cache
 EELAYER 30 0
 EELAYER END
@@
 $0000 - $7EFF\n$7F60 - $7F7F\n$7F80 - $7F9F\n$7FA0 - $7FBF\n$7FC0 - $7FDF\n$7FE0 - $7FFF\n$8000 - $FFFF
 $Comp
-L Oscillator:SG-8002CA X1
+L pluto-rescue:SG-8002CA-Oscillator X1
 U 1 1 5D6922F2
 P 4350 6450
+AR Path="/5D6922F2" Ref="X1"  Part="1"
+AR Path="/58D589A4/5D6922F2" Ref="X1"  Part="1"
 F 0 "X1" H 4175 6700 50  0000 L CNN
 F 1 "16MHz" H 4375 6200 50  0000 L CNN
@@
 Wire Wire Line
 	1125 6000 1675 6000
-Wire Bus Line
-	7375 1025 7375 2025
 $Comp
 L power:GND #PWR0102
@@
 $EndComp
 Connection ~ 1675 6000
+Wire Bus Line
+	7375 1025 7375 2025
 $EndSCHEMATC

Commit message: small updates
Connections:
- net GND: now also Q1.3 (E); no longer Q1.1 (C)
- net ~NMI: now also Q1.1 (C); no longer Q1.3 (E)
Changed lines of the file:
@@
 F 3 "~" H 2650 5050 50  0001 C CNN
 	1    2650 5050
-	-1   0    0    1
+	-1   0    0    -1
 $EndComp
 $Comp
@@
 P 2850 5050
 F 0 "#PWR023" H 2850 4900 50  0001 C CNN
-F 1 "VCC" H 2867 5223 50  0000 C CNN
+F 1 "VCC" H 2850 5000 50  0000 C CNN
 F 2 "" H 2850 5050 50  0001 C CNN
 F 3 "" H 2850 5050 50  0001 C CNN
